Commit message: vhacd for pybullet

File: data/urdf/test/robot.urdf (robot description, URDF)
Before this commit: robot robot, 13 links, 12 joints
Links:
- link 12: mass 0.08730556878781262 -> 0.09918068248396092
- link 9: mass 0.08730556878781262 -> 0.09918068248396095

Commit message: renames

File: data/urdf/test/robot.urdf (robot description, URDF)
Before this commit: robot robot, 13 links, 12 joints
Links:
- link 0: mass 0.6619871640245176 -> 0.6565158606563684
- link 1: mass 0.07174383694960038 -> 0.07174383694960039
- link 10: mass 0.07174383694960038 -> 0.07174383694960039
- link 12: mass 0.09918068248396092 -> 0.10541283606355728
- link 4: mass 0.07174383694960038 -> 0.07174383694960039
- link 7: mass 0.07174383694960038 -> 0.07174383694960039
- link 9: mass 0.09918068248396095 -> 0.10541283606355728
Joints:
- joint 0,1: limit effort=11 velocity=51 -> lower=-3.141592653589793 upper=3.141592653589793; origin xyz=0.07 0.10200000000000001 0.0 rpy=1.5707963267948966 0.0 1.5707963267948966 -> xyz=0.07 0.107 0.0 rpy=1.5707963267948966 0.0 1.5707963267948966
- joint 0,10: limit effort=11 velocity=51 -> lower=-3.141592653589793 upper=3.141592653589793; origin xyz=-0.17500000000000002 -0.025 0.0 rpy=-1.5707963267948966 0.0 -1.5707963267948966 -> xyz=-0.17500000000000002 -0.03 0.0 rpy=-1.5707963267948966 0.0 -1.5707963267948966
- joint 0,4: limit effort=11 velocity=51 -> lower=-3.141592653589793 upper=3.141592653589793; origin xyz=0.07 -0.10200000000000001 0.0 rpy=-1.5707963267948966 0.0 -1.5707963267948966 -> xyz=0.07 -0.107 0.0 rpy=-1.5707963267948966 0.0 -1.5707963267948966
- joint 0,7: limit effort=11 velocity=51 -> lower=-3.141592653589793 upper=3.141592653589793; origin xyz=-0.17500000000000002 0.025 0.0 rpy=1.5707963267948966 0.0 1.5707963267948966 -> xyz=-0.17500000000000002 0.03 0.0 rpy=1.5707963267948966 0.0 1.5707963267948966
- joint 1,2: limit effort=11 velocity=51 -> lower=-1.7453292519943295 upper=1.7453292519943295; origin xyz=0.07100000000000001 0.0 0.0 rpy=1.5707963267948966 0.0 -1.5707963267948966 -> xyz=0.066 0.0 0.0 rpy=1.5707963267948966 0.0 -1.5707963267948966
- joint 10,11: limit effort=11 velocity=51 -> lower=-1.7453292519943295 upper=1.7453292519943295; origin xyz=0.07100000000000001 0.0 0.0 rpy=-1.5707963267948966 0.0 1.5707963267948966 -> xyz=0.066 0.0 0.0 rpy=-1.5707963267948966 0.0 1.5707963267948966
- joint 11,12: limit effort=11 velocity=51 -> lower=-1.5707963267948966 upper=1.5707963267948966
- joint 2,3: limit effort=11 velocity=51 -> lower=-1.5707963267948966 upper=1.5707963267948966
- joint 4,5: limit effort=11 velocity=51 -> lower=-1.7453292519943295 upper=1.7453292519943295; origin xyz=0.07100000000000001 0.0 0.0 rpy=-1.5707963267948966 0.0 1.5707963267948966 -> xyz=0.066 0.0 0.0 rpy=-1.5707963267948966 0.0 1.5707963267948966
- joint 5,6: limit effort=11 velocity=51 -> lower=-1.5707963267948966 upper=1.5707963267948966
- joint 7,8: limit effort=11 velocity=51 -> lower=-1.7453292519943295 upper=1.7453292519943295; origin xyz=0.07100000000000001 0.0 0.0 rpy=1.5707963267948966 0.0 -1.5707963267948966 -> xyz=0.066 0.0 0.0 rpy=1.5707963267948966 0.0 -1.5707963267948966
- joint 8,9: limit effort=11 velocity=51 -> lower=-1.5707963267948966 upper=1.5707963267948966

Commit message: checkpoint

File: data/urdf/test/robot.urdf (robot description, URDF)
Before this commit: robot robot, 13 links, 12 joints
Links:
- link 12: mass 0.10541283606355728 -> 0.10069859040694298
- link 9: mass 0.10541283606355728 -> 0.10069859040694298

Commit message: checkpoint

File: data/urdf/test/robot.urdf (robot description, URDF)
Before this commit: robot robot, 13 links, 12 joints
Links:
- link 12: mass 0.10069859040694298 -> 0.09559312013020987
- link 9: mass 0.10069859040694298 -> 0.09559312013020987

Commit message: modified reward

File: data/urdf/test/robot.urdf (robot description, URDF)
Before this commit: robot robot, 13 links, 12 joints
Links:
- link 12: mass 0.09559312013020987 -> 0.08353239408929022
- link 9: mass 0.09559312013020987 -> 0.08353239408929022

Commit message: replay buffer Emphasizing Recent Experience
ref: https://arxiv.org/abs/1906.04009
Boosting Soft Actor-Critic: Emphasizing Recent Experience without Forgetting the Past

File: data/urdf/test/robot.urdf (robot description, URDF)
Before this commit: robot robot, 13 links, 12 joints
Links:
- link 12: mass 0.08353239408929022 -> 0.07775423696419895
- link 9: mass 0.08353239408929022 -> 0.07775423696419895
