Commit message: modified robot model

File: data/urdf/12dof/robot.urdf (robot description, URDF)
Before this commit: robot robot, 13 links, 12 joints
Links:
- link 0: mass 0.6565158606563684 -> 0.6982204026089079
- link 12: mass 0.07775423696419895 -> 0.08532948636481331
- link 9: mass 0.07775423696419895 -> 0.08532948636481333

Commit message: modified feet

File: data/urdf/12dof/robot.urdf (robot description, URDF)
Before this commit: robot robot, 13 links, 12 joints
Links:
- link 12: mass 0.08532948636481331 -> 0.07811450734720533
- link 9: mass 0.08532948636481333 -> 0.07811450734720533

Commit message: smaller feet

File: data/urdf/12dof/robot.urdf (robot description, URDF)
Before this commit: robot robot, 13 links, 12 joints
Links:
- link 12: mass 0.07811450734720533 -> 0.08034452961093837
- link 9: mass 0.07811450734720533 -> 0.08034452961093837

Commit message: modified feet

File: data/urdf/12dof/robot.urdf (robot description, URDF)
Before this commit: robot robot, 13 links, 12 joints
Links:
- link 12: mass 0.08034452961093837 -> 0.0778070440712388
- link 9: mass 0.08034452961093837 -> 0.0778070440712388

Commit message: hand

File: data/urdf/12dof/robot.urdf (robot description, URDF)
Before this commit: robot robot, 13 links, 12 joints
Links:
- link 12: mass 0.0778070440712388 -> 0.07228479126379891
- link 3: mass 0.07279808599447314 -> 0.06648163941481205
- link 6: mass 0.07279808599447314 -> 0.06648163941481205
- link 9: mass 0.0778070440712388 -> 0.07228479126379891

Commit message: spring compliance, modified robot

File: data/urdf/12dof/robot.urdf (robot description, URDF)
Before this commit: robot robot, 13 links, 12 joints
Links:
- link 12: mass 0.07228479126379891 -> 0.07441012134499128
- link 3: mass 0.06648163941481205 -> 0.06983417080751726
- link 6: mass 0.06648163941481205 -> 0.06983417080751726
- link 9: mass 0.07228479126379891 -> 0.07441012134499125

Commit message: biped

File: data/urdf/12dof/robot.urdf (robot description, URDF)
Before this commit: robot robot, 13 links, 12 joints
Links:
- link 12: mass 0.07441012134499128 -> 0.0767626626962517
- link 3: mass 0.06983417080751726 -> 0.07318680108662914
- link 6: mass 0.06983417080751726 -> 0.07318680108662914
- link 9: mass 0.07441012134499125 -> 0.0767626626962517

Commit message: manual stepping

File: data/urdf/12dof/robot.urdf (robot description, URDF)
Before this commit: robot robot, 13 links, 12 joints
Links:
- link 0: mass 0.6982204026089079 -> 0.6139850203204843
- link 1: mass 0.07174383694960039 -> 0.07269017067211427
- link 10: mass 0.07174383694960039 -> 0.07269017067211427
- link 11: mass 0.10679863001648698 -> 0.09857950140569696
- link 12: mass 0.0767626626962517 -> 0.06025949243310835
- link 2: mass 0.10679863001648698 -> 0.09857950140569696
- link 3: mass 0.07318680108662914 -> 0.05961127877722497
- link 4: mass 0.07174383694960039 -> 0.07269017067211427
- link 5: mass 0.10679863001648698 -> 0.09857950140569696
- link 6: mass 0.07318680108662914 -> 0.05961127877722497
- link 7: mass 0.07174383694960039 -> 0.07269017067211427
- link 8: mass 0.10679863001648698 -> 0.09857950140569696
- link 9: mass 0.0767626626962517 -> 0.06025949243310835
Joints:
- joint 0,1: origin xyz=0.07 0.107 0.0 rpy=1.5707963267948966 0.0 1.5707963267948966 -> xyz=0.048 0.107 0.0 rpy=1.5707963267948966 0.0 1.5707963267948966
- joint 0,10: origin xyz=-0.17500000000000002 -0.03 0.0 rpy=-1.5707963267948966 0.0 -1.5707963267948966 -> xyz=-0.153 -0.03 0.0 rpy=-1.5707963267948966 0.0 -1.5707963267948966
- joint 0,4: origin xyz=0.07 -0.107 0.0 rpy=-1.5707963267948966 0.0 -1.5707963267948966 -> xyz=0.048 -0.107 0.0 rpy=-1.5707963267948966 0.0 -1.5707963267948966
- joint 0,7: origin xyz=-0.17500000000000002 0.03 0.0 rpy=1.5707963267948966 0.0 1.5707963267948966 -> xyz=-0.153 0.03 0.0 rpy=1.5707963267948966 0.0 1.5707963267948966
- joint 11,12: origin xyz=0.0 0.0 -0.14300000000000002 rpy=0.0 0.0 1.5707963267948963 -> xyz=0.0 0.0 -0.13 rpy=0.0 0.0 1.5707963267948963
- joint 2,3: origin xyz=0.0 0.0 -0.14300000000000002 rpy=0.0 0.0 -1.5707963267948963 -> xyz=0.0 0.0 -0.13 rpy=0.0 0.0 -1.5707963267948963
- joint 5,6: origin xyz=0.0 0.0 -0.14300000000000002 rpy=0.0 0.0 1.5707963267948963 -> xyz=0.0 0.0 -0.13 rpy=0.0 0.0 1.5707963267948963
- joint 8,9: origin xyz=0.0 0.0 -0.14300000000000002 rpy=0.0 0.0 -1.5707963267948963 -> xyz=0.0 0.0 -0.13 rpy=0.0 0.0 -1.5707963267948963
