Commit message: updated v11 robot

File: robot/v11/urdf/robot.urdf (robot description, URDF)
Before this commit: robot robot, 13 links, 12 joints
Links:
- link 0: mass 0.600805171853325 -> 0.6162799829535238
- link 10: mass 0.07269017067211427 -> 0.1338270472340628
- link 11: mass 0.09857950140569696 -> 0.0921671006538613
- link 12: mass 0.07438935151938421 -> 0.05398256592708953
- link 7: mass 0.07269017067211427 -> 0.1338270472340628
- link 8: mass 0.09857950140569696 -> 0.0921671006538613
- link 9: mass 0.07438935151938421 -> 0.053982565927089526
Joints:
- joint 0,10: origin xyz=-0.153 -0.03 0.0 rpy=-1.5707963267948966 0.0 -1.5707963267948966 -> xyz=-0.153 -0.029 0.0 rpy=-1.5707963267948966 0.0 -1.5707963267948966
- joint 0,7: origin xyz=-0.153 0.03 0.0 rpy=1.5707963267948966 0.0 1.5707963267948966 -> xyz=-0.153 0.029 0.0 rpy=1.5707963267948966 0.0 1.5707963267948966
- joint 10,11: origin xyz=0.066 0.0 0.0 rpy=-1.5707963267948966 0.0 1.5707963267948966 -> xyz=0.051000000000000004 0.0 -0.1 rpy=0.0 0.0 0.0
- joint 11,12: origin xyz=0.0 0.0 -0.13 rpy=0.0 0.0 1.5707963267948966 -> xyz=0.0 0.0 -0.112 rpy=0.0 0.0 0.0
- joint 7,8: origin xyz=0.066 0.0 0.0 rpy=1.5707963267948966 0.0 -1.5707963267948966 -> xyz=0.051000000000000004 0.0 -0.1 rpy=0.0 0.0 0.0
- joint 8,9: origin xyz=0.0 0.0 -0.13 rpy=0.0 0.0 -1.5707963267948966 -> xyz=0.0 0.0 -0.112 rpy=0.0 0.0 0.0
